Commit message: visual update

File: lab_2/urdf/dynamic.urdf.xacro (robot description, xacro)
@@ -70,10 +70,10 @@
     <child link="i2"/>
 		<axis xyz="0 0 1"/>
-    <origin rpy = "1.57 -0.0 1.57 " xyz= "0.0 0.0 1.0"/>
+    <origin rpy = "1.57 -0.0 1.57 " xyz= "1.0 0.0 0.0"/>
   </joint>
 	<link name="i3">
 		<visual>
 			<geometry>
-				<cylinder length="${params['i3_h']}" radius="${params['i3_r']}"/>
+				<cylinder length="${params['i3_h']}" radius=" ${params['i3_r']}"/>
 			</geometry>
 			<origin rpy= "0 0 0" xyz="0.0 0 0"/>
@@ -90,9 +90,33 @@
     </inertial>
 	</link>
-	<joint name="i_3" type="continuous">
+	<joint name="i_3" type="revolute">
     <parent link="i2"/>
     <child link="i3"/>
+		<limit effort="100.0" lower="-1.57" upper="1.57" velocity="0.5"/>
 		<axis xyz="0 0 1"/>
-    <origin rpy = "1.57 -0.0 1.57 " xyz= "0.0 0.0 1.0"/>
+    <origin rpy = "1.57 -0.0 1.57 " xyz= "1.0 0.0 0.0"/>
+  </joint>
+	<link name="tool">
+		<visual>
+			<geometry>
+				<box size="${params['tool_a']} ${params['tool_b']} ${params['tool_c']}"/>
+			</geometry>
+			<origin rpy= "0 0 0" xyz="0.0 0 0"/>
+			<material name="blue"/>
+		</visual>
+	<collision>
+      <geometry>
+        <box size="${params['tool_a']} ${params['tool_b']} ${params['tool_c']}"/>
+      </geometry>
+    </collision>
+    <inertial>
+      <mass value="10"/>
+      <inertia ixx="1.0" ixy="0.0" ixz="0.0" iyy="1.0" iyz="0.0" izz="1.0"/>
+    </inertial>
+	</link>
+	<joint name="tool_joint" type="fixed">
+    <parent link="i3"/>
+    <child link="tool"/>
+    <origin rpy = "0.0 0.0 0.0" xyz= "0.0 0.5 0.0"/>
   </joint>
 </robot>

File: lab_2/urdf/dynamic2.urdf.xacro (robot description, xacro)
@@ -1,5 +1,5 @@
 <?xml version="1.0"?>
 <robot name="visual" xmlns:xacro="https://ros.org/wiki/xacro">
-	<xacro:property name="params" value="${load_yaml('../yaml/params.yaml')}"/>
+	<xacro:property name="params" value="${load_yaml('../yaml/params2.yaml')}"/>
 	<material name="blue">
     <color rgba="0 0 0.8 1"/>
@@ -20,5 +20,5 @@
 		<collision>
       <geometry>
-        <cylinder length="0.05" radius="0.2"/>
+        <cylinder length="0.4" radius="0.2"/>
       </geometry>
     </collision>
@@ -27,5 +27,5 @@
     <visual>
       <geometry>
-        <cylinder length="${params['i1_h']}" radius="${params['i1_r']}"/>
+        <box size="${params['i1_a']} ${params['i1_b']} ${params['i1_c']}"/>
       </geometry>
       <origin rpy="0 0 0 " xyz="0.0 0 0"/>
@@ -34,5 +34,5 @@
 		<collision>
       <geometry>
-        <cylinder length="${params['i1_h']}" radius="${params['i1_r']}"/>
+        <box size="${params['i1_a']} ${params['i1_c']} ${params['i1_c']}"/>
       </geometry>
     </collision>
@@ -42,7 +42,8 @@
     </inertial>
   </link>
-	<joint name="i_1" type="fixed">
+	<joint name="i_1" type="continuous">
     <parent link="base_link"/>
     <child link="i1"/>
+		<axis xyz="0 0 1"/>
     <origin rpy = "0.0 -0.0 0.0" xyz= "0 0 1.0"/>
   </joint>
@@ -53,5 +54,5 @@
 			</geometry>
 			<origin rpy= "0 0 0" xyz="0.0 0 0"/>
-			<material name="white"/>
+			<material name="black"/>
 		</visual>
 	<collision>
@@ -65,20 +66,21 @@
     </inertial>
 	</link>
-	<joint name="i_2" type="fixed">
+	<joint name="i_2" type="continuous">
     <parent link="i1"/>
     <child link="i2"/>
-    <origin rpy = "1.57 -0.0 1.57 " xyz= "0.0 0.0 1.0"/>
+		<axis xyz="0 0 1"/>
+    <origin rpy = "1.57 -0.0 1.57 " xyz= "1.0 0.0 0.0"/>
   </joint>
 	<link name="i3">
 		<visual>
 			<geometry>
-				<box size="${params['i3_a']} ${params['i3_b']} ${params['i3_c']}"/>
+				<cylinder length="${params['i3_h']}" radius=" ${params['i3_r']}"/>
 			</geometry>
 			<origin rpy= "0 0 0" xyz="0.0 0 0"/>
-			<material name="black"/>
+			<material name="white"/>
 		</visual>
 	<collision>
       <geometry>
-        <box size="${params['i3_a']} ${params['i3_b']} ${params['i3_c']}"/>
+        <cylinder length="${params['i3_h']}" radius="${params['i3_r']}"/>
       </geometry>
     </collision>
@@ -88,8 +90,33 @@
     </inertial>
 	</link>
-	<joint name="i_3" type="fixed">
+	<joint name="i_3" type="revolute">
     <parent link="i2"/>
     <child link="i3"/>
-    <origin rpy = "1.57 -0.0 1.57 " xyz= "0.0 0.0 1.0"/>
+		<limit effort="100.0" lower="-1.57" upper="1.57" velocity="0.5"/>
+		<axis xyz="0 0 1"/>
+    <origin rpy = "1.57 -0.0 1.57 " xyz= "1.0 0.0 0.0"/>
+  </joint>
+	<link name="tool">
+		<visual>
+			<geometry>
+				<box size="${params['tool_a']} ${params['tool_b']} ${params['tool_c']}"/>
+			</geometry>
+			<origin rpy= "0 0 0" xyz="0.0 0 0"/>
+			<material name="blue"/>
+		</visual>
+	<collision>
+      <geometry>
+        <box size="${params['tool_a']} ${params['tool_b']} ${params['tool_c']}"/>
+      </geometry>
+    </collision>
+    <inertial>
+      <mass value="10"/>
+      <inertia ixx="1.0" ixy="0.0" ixz="0.0" iyy="1.0" iyz="0.0" izz="1.0"/>
+    </inertial>
+	</link>
+	<joint name="tool_joint" type="fixed">
+    <parent link="i3"/>
+    <child link="tool"/>
+    <origin rpy = "0.0 0.0 0.0" xyz= "0.0 0.5 0.0"/>
   </joint>
 </robot>

Commit message: final version

File: lab_2/urdf/dynamic.urdf.xacro (robot description, xacro)
@@ -2,4 +2,5 @@
 <robot name="visual" xmlns:xacro="https://ros.org/wiki/xacro">
 	<xacro:property name="params" value="${load_yaml('../yaml/params.yaml')}"/>
+	<xacro:property name="param" value="${load_yaml('../yaml/urdf.yaml')}"/>
 	<material name="blue">
     <color rgba="0 0 0.8 1"/>
@@ -13,12 +14,14 @@
 	<link name="base_link">
     <visual>
+			<origin xyz = "0 0 ${params['base_h']/2}"/>
       <geometry>
-        <cylinder length="0.05" radius="0.2"/>
+        <cylinder length="${params['base_h']}" radius="${params['base_r']}"/>
       </geometry>
       <material name="white"/>
     </visual>
 		<collision>
+			<origin xyz = "0 0 ${params['base_h']/2}"/>
       <geometry>
-        <cylinder length="0.05" radius="0.2"/>
+        <cylinder length="${params['base_h']}" radius="${params['base_r']}"/>
       </geometry>
     </collision>
@@ -27,12 +30,13 @@
     <visual>
       <geometry>
-        <cylinder length="${params['i1_h']}" radius="${params['i1_r']}"/>
+        <box size="${params['i1_a']} ${params['i1_b']} ${params['d1']}"/>
       </geometry>
-      <origin rpy="0 0 0 " xyz="0.0 0 0"/>
+      <origin rpy="0 0 0 " xyz="0.0 0 ${params['d1']/2}"/>
       <material name="blue"/>
     </visual>
 		<collision>
+			<origin rpy="0 0 0 " xyz="0.0 0 ${params['d1']/2}"/>
       <geometry>
-        <cylinder length="${params['i1_h']}" radius="${params['i1_r']}"/>
+        <box size="${params['i1_a']} ${params['i1_b']} ${params['d1']}"/>
       </geometry>
     </collision>
@@ -46,17 +50,18 @@
     <child link="i1"/>
 		<axis xyz="0 0 1"/>
-    <origin rpy = "0.0 -0.0 0.0" xyz= "0 0 1.0"/>
+    <origin rpy = "${param['i_1']['joint_rpy']}" xyz= "0 0 ${params['base_h']}"/>
   </joint>
 	<link name="i2">
 		<visual>
 			<geometry>
-				<cylinder length="${params['i2_h']}" radius="${params['i2_r']}"/>
+				<cylinder length="${params['d2']-params['i1_b']}" radius="${params['i2_r']}"/>
 			</geometry>
-			<origin rpy= "0 0 0" xyz="0.0 0 0"/>
+			<origin rpy="0 0 0 " xyz="0.0 0 ${params['d2']/2}"/>
 			<material name="black"/>
 		</visual>
 	<collision>
+			<origin rpy="0 0 0 " xyz="0.0 0 ${params['d2']/2}"/>
       <geometry>
-        <cylinder length="${params['i2_h']}" radius="${params['i2_r']}"/>
+        <cylinder length="${params['d2']}" radius="${params['i2_r']}"/>
       </geometry>
     </collision>
@@ -70,17 +75,18 @@
     <child link="i2"/>
 		<axis xyz="0 0 1"/>
-    <origin rpy = "1.57 -0.0 1.57 " xyz= "1.0 0.0 0.0"/>
+    <origin rpy = "${param['i_2']['joint_rpy']}" xyz= "${param['i_2']['joint_xyz']}"/>
   </joint>
 	<link name="i3">
 		<visual>
 			<geometry>
-				<cylinder length="${params['i3_h']}" radius=" ${params['i3_r']}"/>
+				<cylinder length="${params['d3']-params['i2_r']}" radius=" ${params['i3_r']}"/>
 			</geometry>
-			<origin rpy= "0 0 0" xyz="0.0 0 0"/>
+			<origin rpy="0 0 0 " xyz="0.0 0 ${params['d3']/2}"/>
 			<material name="white"/>
 		</visual>
 	<collision>
+			<origin rpy="0 0 0 " xyz="0.0 0 ${params['d3']/2}"/>
       <geometry>
-        <cylinder length="${params['i3_h']}" radius="${params['i3_r']}"/>
+        <cylinder length="${params['d3']}" radius="${params['i3_r']}"/>
       </geometry>
     </collision>
@@ -90,20 +96,20 @@
     </inertial>
 	</link>
-	<joint name="i_3" type="revolute">
+	<joint name="i_3" type="continuous">
     <parent link="i2"/>
     <child link="i3"/>
-		<limit effort="100.0" lower="-1.57" upper="1.57" velocity="0.5"/>
 		<axis xyz="0 0 1"/>
-    <origin rpy = "1.57 -0.0 1.57 " xyz= "1.0 0.0 0.0"/>
+    <origin rpy = "${param['i_3']['joint_rpy']}" xyz= "${param['i_3']['joint_xyz']}"/>
   </joint>
 	<link name="tool">
 		<visual>
 			<geometry>
-				<box size="${params['tool_a']} ${params['tool_b']} ${params['tool_c']}"/>
+				<box size="${params['tool_a']} ${params['tool_b']-params['i3_r']} ${params['tool_c']}"/>
 			</geometry>
-			<origin rpy= "0 0 0" xyz="0.0 0 0"/>
+			<origin rpy= "0 0 0" xyz="0.0 ${params['tool_b']/2} 0"/>
 			<material name="blue"/>
 		</visual>
 	<collision>
+			<origin rpy= "0 0 0" xyz="0.0 ${params['tool_b']/2} 0 "/>
       <geometry>
         <box size="${params['tool_a']} ${params['tool_b']} ${params['tool_c']}"/>
@@ -118,5 +124,5 @@
     <parent link="i3"/>
     <child link="tool"/>
-    <origin rpy = "0.0 0.0 0.0" xyz= "0.0 0.5 0.0"/>
+    <origin rpy = "0.0 0.0 0.0" xyz= "0.0 0.0 ${params['d3']}"/>
   </joint>
 </robot>

File: lab_2/urdf/static.urdf.xacro (robot description, xacro)
@@ -1,5 +1,6 @@
 <?xml version="1.0"?>
 <robot name="visual" xmlns:xacro="https://ros.org/wiki/xacro">
-	<xacro:property name="params" value="${load_yaml('../yaml/params.yaml')}"/>
+	<xacro:property name="params" value="${load_yaml('../yaml/params2.yaml')}"/>
+	<xacro:property name="param" value="${load_yaml('../yaml/urdf.yaml')}"/>
 	<material name="blue">
     <color rgba="0 0 0.8 1"/>
@@ -13,12 +14,14 @@
 	<link name="base_link">
     <visual>
+			<origin xyz = "0 0 ${params['base_h']/2}"/>
       <geometry>
-        <cylinder length="0.2" radius="0.2"/>
+        <cylinder length="${params['base_h']}" radius="${params['base_r']}"/>
       </geometry>
       <material name="white"/>
     </visual>
 		<collision>
+			<origin xyz = "0 0 ${params['base_h']/2}"/>
       <geometry>
-        <cylinder length="0.05" radius="0.2"/>
+        <cylinder length="${params['base_h']}" radius="${params['base_r']}"/>
       </geometry>
     </collision>
@@ -27,12 +30,13 @@
     <visual>
       <geometry>
-        <cylinder length="${params['i1_h']}" radius="${params['i1_r']}"/>
+        <box size="${params['i1_a']} ${params['i1_b']} ${params['d1']}"/>
       </geometry>
-      <origin rpy="0 0 0 " xyz="0.0 0 0"/>
+      <origin rpy="0 0 0 " xyz="0.0 0 ${params['d1']/2}"/>
       <material name="blue"/>
     </visual>
 		<collision>
+			<origin rpy="0 0 0 " xyz="0.0 0 ${params['d1']/2}"/>
       <geometry>
-        <cylinder length="${params['i1_h']}" radius="${params['i1_r']}"/>
+        <box size="${params['i1_a']} ${params['i1_b']} ${params['d1']}"/>
       </geometry>
     </collision>
@@ -45,17 +49,19 @@
     <parent link="base_link"/>
     <child link="i1"/>
-    <origin rpy = "0.0 -0.0 0.0" xyz= "0 0 1.0"/>
+		<axis xyz="0 0 1"/>
+    <origin rpy = "${param['i_1']['joint_rpy']}" xyz= "0 0 ${params['base_h']}"/>
   </joint>
 	<link name="i2">
 		<visual>
 			<geometry>
-				<cylinder length="${params['i2_h']}" radius="${params['i2_r']}"/>
+				<cylinder length="${params['d2']-params['i1_b']}" radius="${params['i2_r']}"/>
 			</geometry>
-			<origin rpy= "0 0 0" xyz="0.0 0 0"/>
-			<material name="white"/>
+			<origin rpy="0 0 0 " xyz="0.0 0 ${params['d2']/2}"/>
+			<material name="black"/>
 		</visual>
 	<collision>
+			<origin rpy="0 0 0 " xyz="0.0 0 ${params['d2']/2}"/>
       <geometry>
-        <cylinder length="${params['i2_h']}" radius="${params['i2_r']}"/>
+        <cylinder length="${params['d2']}" radius="${params['i2_r']}"/>
       </geometry>
     </collision>
@@ -68,17 +74,19 @@
     <parent link="i1"/>
     <child link="i2"/>
-    <origin rpy = "1.57 -0.0 1.57 " xyz= "0.0 0.0 1.0"/>
+		<axis xyz="0 0 1"/>
+    <origin rpy = "${param['i_2']['joint_rpy']}" xyz= "${param['i_2']['joint_xyz']}"/>
   </joint>
 	<link name="i3">
 		<visual>
 			<geometry>
-				<box size="${params['i3_a']} ${params['i3_b']} ${params['i3_c']}"/>
+				<cylinder length="${params['d3']-params['i2_r']}" radius=" ${params['i3_r']}"/>
 			</geometry>
-			<origin rpy= "0 0 0" xyz="0.0 0 0"/>
-			<material name="black"/>
+			<origin rpy="0 0 0 " xyz="0.0 0 ${params['d3']/2}"/>
+			<material name="white"/>
 		</visual>
 	<collision>
+			<origin rpy="0 0 0 " xyz="0.0 0 ${params['d3']/2}"/>
       <geometry>
-        <box size="${params['i3_a']} ${params['i3_b']} ${params['i3_c']}"/>
+        <cylinder length="${params['d3']}" radius="${params['i3_r']}"/>
       </geometry>
     </collision>
@@ -91,5 +99,30 @@
     <parent link="i2"/>
     <child link="i3"/>
-    <origin rpy = "1.57 -0.0 1.57 " xyz= "0.0 0.0 1.0"/>
+		<axis xyz="0 0 1"/>
+    <origin rpy = "${param['i_3']['joint_rpy']}" xyz= "${param['i_3']['joint_xyz']}"/>
+  </joint>
+	<link name="tool">
+		<visual>
+			<geometry>
+				<box size="${params['tool_a']} ${params['tool_b']-params['i3_r']} ${params['tool_c']}"/>
+			</geometry>
+			<origin rpy= "0 0 0" xyz="0.0 ${params['tool_b']/2} 0"/>
+			<material name="blue"/>
+		</visual>
+	<collision>
+			<origin rpy= "0 0 0" xyz="0.0 ${params['tool_b']/2} 0 "/>
+      <geometry>
+        <box size="${params['tool_a']} ${params['tool_b']} ${params['tool_c']}"/>
+      </geometry>
+    </collision>
+    <inertial>
+      <mass value="10"/>
+      <inertia ixx="1.0" ixy="0.0" ixz="0.0" iyy="1.0" iyz="0.0" izz="1.0"/>
+    </inertial>
+	</link>
+	<joint name="tool_joint" type="fixed">
+    <parent link="i3"/>
+    <child link="tool"/>
+    <origin rpy = "0.0 0.0 0.0" xyz= "0.0 0.0 ${params['d3']}"/>
   </joint>
 </robot>
