Commit message: tidy up urdf files

File: lab_2/urdf/dynamic.urdf.xacro (robot description, xacro)
@@ -4,52 +4,52 @@
 	<xacro:property name="param" value="${load_yaml('../yaml/urdf.yaml')}"/>
 	<material name="blue">
-    <color rgba="0 0 0.8 1"/>
-  </material>
-  <material name="black">
-    <color rgba="0 0 0 1"/>
-  </material>
-  <material name="white">
-    <color rgba="1 1 1 1"/>
-  </material>
+		<color rgba="0 0 0.8 1"/>
+	</material>
+	<material name="black">
+		<color rgba="0 0 0 1"/>
+	</material>
+	<material name="white">
+		<color rgba="1 1 1 1"/>
+	</material>
 	<link name="base_link">
-    <visual>
+		<visual>
 			<origin xyz = "0 0 ${params['base_h']/2}"/>
-      <geometry>
-        <cylinder length="${params['base_h']}" radius="${params['base_r']}"/>
-      </geometry>
-      <material name="white"/>
-    </visual>
+			<geometry>
+				<cylinder length="${params['base_h']}" radius="${params['base_r']}"/>
+			</geometry>
+			<material name="white"/>
+		</visual>
 		<collision>
 			<origin xyz = "0 0 ${params['base_h']/2}"/>
-      <geometry>
-        <cylinder length="${params['base_h']}" radius="${params['base_r']}"/>
-      </geometry>
-    </collision>
-  </link>
+			<geometry>
+				<cylinder length="${params['base_h']}" radius="${params['base_r']}"/>
+			</geometry>
+		</collision>
+  	</link>
 	<link name="i1">
-    <visual>
-      <geometry>
-        <box size="${params['i1_a']} ${params['i1_b']} ${params['d1']}"/>
-      </geometry>
-      <origin rpy="0 0 0 " xyz="0.0 0 ${params['d1']/2}"/>
-      <material name="blue"/>
-    </visual>
+		<visual>
+			<geometry>
+				<box size="${params['i1_a']} ${params['i1_b']} ${params['d1']}"/>
+			</geometry>
+			<origin rpy="0 0 0 " xyz="0.0 0 ${params['d1']/2}"/>
+			<material name="blue"/>
+		</visual>
 		<collision>
 			<origin rpy="0 0 0 " xyz="0.0 0 ${params['d1']/2}"/>
-      <geometry>
-        <box size="${params['i1_a']} ${params['i1_b']} ${params['d1']}"/>
-      </geometry>
-    </collision>
-    <inertial>
-      <mass value="10"/>
-      <inertia ixx="1.0" ixy="0.0" ixz="0.0" iyy="1.0" iyz="0.0" izz="1.0"/>
-    </inertial>
-  </link>
+			<geometry>
+				<box size="${params['i1_a']} ${params['i1_b']} ${params['d1']}"/>
+			</geometry>
+		</collision>
+		<inertial>
+			<mass value="10"/>
+			<inertia ixx="1.0" ixy="0.0" ixz="0.0" iyy="1.0" iyz="0.0" izz="1.0"/>
+		</inertial>
+	</link>
 	<joint name="i_1" type="continuous">
-    <parent link="base_link"/>
-    <child link="i1"/>
+		<parent link="base_link"/>
+		<child link="i1"/>
 		<axis xyz="0 0 1"/>
-    <origin rpy = "${param['i_1']['joint_rpy']}" xyz= "0 0 ${params['base_h']}"/>
-  </joint>
+		<origin rpy = "${param['i_1']['joint_rpy']}" xyz= "0 0 ${params['base_h']}"/>
+	</joint>
 	<link name="i2">
 		<visual>
@@ -60,21 +60,21 @@
 			<material name="black"/>
 		</visual>
-	<collision>
+		<collision>
 			<origin rpy="0 0 0 " xyz="0.0 0 ${params['d2']/2}"/>
-      <geometry>
-        <cylinder length="${params['d2']}" radius="${params['i2_r']}"/>
-      </geometry>
-    </collision>
-    <inertial>
-      <mass value="10"/>
-      <inertia ixx="1.0" ixy="0.0" ixz="0.0" iyy="1.0" iyz="0.0" izz="1.0"/>
-    </inertial>
+			<geometry>
+				<cylinder length="${params['d2']}" radius="${params['i2_r']}"/>
+			</geometry>
+		</collision>
+		<inertial>
+			<mass value="10"/>
+			<inertia ixx="1.0" ixy="0.0" ixz="0.0" iyy="1.0" iyz="0.0" izz="1.0"/>
+		</inertial>
 	</link>
 	<joint name="i_2" type="continuous">
-    <parent link="i1"/>
-    <child link="i2"/>
+		<parent link="i1"/>
+		<child link="i2"/>
 		<axis xyz="0 0 1"/>
-    <origin rpy = "${param['i_2']['joint_rpy']}" xyz= "${param['i_2']['joint_xyz']}"/>
-  </joint>
+		<origin rpy = "${param['i_2']['joint_rpy']}" xyz= "${param['i_2']['joint_xyz']}"/>
+	</joint>
 	<link name="i3">
 		<visual>
@@ -85,21 +85,21 @@
 			<material name="white"/>
 		</visual>
-	<collision>
+		<collision>
 			<origin rpy="0 0 0 " xyz="0.0 0 ${params['d3']/2}"/>
-      <geometry>
-        <cylinder length="${params['d3']}" radius="${params['i3_r']}"/>
-      </geometry>
-    </collision>
-    <inertial>
-      <mass value="10"/>
-      <inertia ixx="1.0" ixy="0.0" ixz="0.0" iyy="1.0" iyz="0.0" izz="1.0"/>
-    </inertial>
+			<geometry>
+				<cylinder length="${params['d3']}" radius="${params['i3_r']}"/>
+			</geometry>
+		</collision>
+		<inertial>
+			<mass value="10"/>
+			<inertia ixx="1.0" ixy="0.0" ixz="0.0" iyy="1.0" iyz="0.0" izz="1.0"/>
+		</inertial>
 	</link>
 	<joint name="i_3" type="continuous">
-    <parent link="i2"/>
-    <child link="i3"/>
+		<parent link="i2"/>
+		<child link="i3"/>
 		<axis xyz="0 0 1"/>
-    <origin rpy = "${param['i_3']['joint_rpy']}" xyz= "${param['i_3']['joint_xyz']}"/>
-  </joint>
+		<origin rpy = "${param['i_3']['joint_rpy']}" xyz= "${param['i_3']['joint_xyz']}"/>
+	</joint>
 	<link name="tool">
 		<visual>
@@ -110,19 +110,19 @@
 			<material name="blue"/>
 		</visual>
-	<collision>
+		<collision>
 			<origin rpy= "0 0 0" xyz="0.0 ${params['tool_b']/2} 0 "/>
-      <geometry>
-        <box size="${params['tool_a']} ${params['tool_b']} ${params['tool_c']}"/>
-      </geometry>
-    </collision>
-    <inertial>
-      <mass value="10"/>
-      <inertia ixx="1.0" ixy="0.0" ixz="0.0" iyy="1.0" iyz="0.0" izz="1.0"/>
-    </inertial>
+			<geometry>
+				<box size="${params['tool_a']} ${params['tool_b']} ${params['tool_c']}"/>
+			</geometry>
+		</collision>
+		<inertial>
+			<mass value="10"/>
+			<inertia ixx="1.0" ixy="0.0" ixz="0.0" iyy="1.0" iyz="0.0" izz="1.0"/>
+		</inertial>
 	</link>
 	<joint name="tool_joint" type="fixed">
-    <parent link="i3"/>
-    <child link="tool"/>
-    <origin rpy = "0.0 0.0 0.0" xyz= "0.0 0.0 ${params['d3']}"/>
-  </joint>
+		<parent link="i3"/>
+		<child link="tool"/>
+		<origin rpy = "0.0 0.0 0.0" xyz= "0.0 0.0 ${params['d3']}"/>
+	</joint>
 </robot>

File: lab_2/urdf/static.urdf.xacro (robot description, xacro)
@@ -1,55 +1,55 @@
 <?xml version="1.0"?>
 <robot name="visual" xmlns:xacro="https://ros.org/wiki/xacro">
-	<xacro:property name="params" value="${load_yaml('../yaml/params2.yaml')}"/>
+	<xacro:property name="params" value="${load_yaml('../yaml/params.yaml')}"/>
 	<xacro:property name="param" value="${load_yaml('../yaml/urdf.yaml')}"/>
 	<material name="blue">
-    <color rgba="0 0 0.8 1"/>
-  </material>
-  <material name="black">
-    <color rgba="0 0 0 1"/>
-  </material>
-  <material name="white">
-    <color rgba="1 1 1 1"/>
-  </material>
+		<color rgba="0 0 0.8 1"/>
+	</material>
+	<material name="black">
+		<color rgba="0 0 0 1"/>
+	</material>
+	<material name="white">
+		<color rgba="1 1 1 1"/>
+	</material>
 	<link name="base_link">
-    <visual>
+		<visual>
 			<origin xyz = "0 0 ${params['base_h']/2}"/>
-      <geometry>
-        <cylinder length="${params['base_h']}" radius="${params['base_r']}"/>
-      </geometry>
-      <material name="white"/>
-    </visual>
+			<geometry>
+				<cylinder length="${params['base_h']}" radius="${params['base_r']}"/>
+			</geometry>
+			<material name="white"/>
+		</visual>
 		<collision>
 			<origin xyz = "0 0 ${params['base_h']/2}"/>
-      <geometry>
-        <cylinder length="${params['base_h']}" radius="${params['base_r']}"/>
-      </geometry>
-    </collision>
-  </link>
+			<geometry>
+				<cylinder length="${params['base_h']}" radius="${params['base_r']}"/>
+			</geometry>
+		</collision>
+  	</link>
 	<link name="i1">
-    <visual>
-      <geometry>
-        <box size="${params['i1_a']} ${params['i1_b']} ${params['d1']}"/>
-      </geometry>
-      <origin rpy="0 0 0 " xyz="0.0 0 ${params['d1']/2}"/>
-      <material name="blue"/>
-    </visual>
+		<visual>
+			<geometry>
+				<box size="${params['i1_a']} ${params['i1_b']} ${params['d1']}"/>
+			</geometry>
+			<origin rpy="0 0 0 " xyz="0.0 0 ${params['d1']/2}"/>
+			<material name="blue"/>
+		</visual>
 		<collision>
 			<origin rpy="0 0 0 " xyz="0.0 0 ${params['d1']/2}"/>
-      <geometry>
-        <box size="${params['i1_a']} ${params['i1_b']} ${params['d1']}"/>
-      </geometry>
-    </collision>
-    <inertial>
-      <mass value="10"/>
-      <inertia ixx="1.0" ixy="0.0" ixz="0.0" iyy="1.0" iyz="0.0" izz="1.0"/>
-    </inertial>
-  </link>
+			<geometry>
+				<box size="${params['i1_a']} ${params['i1_b']} ${params['d1']}"/>
+			</geometry>
+		</collision>
+		<inertial>
+			<mass value="10"/>
+			<inertia ixx="1.0" ixy="0.0" ixz="0.0" iyy="1.0" iyz="0.0" izz="1.0"/>
+		</inertial>
+	</link>
 	<joint name="i_1" type="fixed">
-    <parent link="base_link"/>
-    <child link="i1"/>
+		<parent link="base_link"/>
+		<child link="i1"/>
 		<axis xyz="0 0 1"/>
-    <origin rpy = "${param['i_1']['joint_rpy']}" xyz= "0 0 ${params['base_h']}"/>
-  </joint>
+		<origin rpy = "${param['i_1']['joint_rpy']}" xyz= "0 0 ${params['base_h']}"/>
+	</joint>
 	<link name="i2">
 		<visual>
@@ -60,21 +60,21 @@
 			<material name="black"/>
 		</visual>
-	<collision>
+		<collision>
 			<origin rpy="0 0 0 " xyz="0.0 0 ${params['d2']/2}"/>
-      <geometry>
-        <cylinder length="${params['d2']}" radius="${params['i2_r']}"/>
-      </geometry>
-    </collision>
-    <inertial>
-      <mass value="10"/>
-      <inertia ixx="1.0" ixy="0.0" ixz="0.0" iyy="1.0" iyz="0.0" izz="1.0"/>
-    </inertial>
+			<geometry>
+				<cylinder length="${params['d2']}" radius="${params['i2_r']}"/>
+			</geometry>
+		</collision>
+		<inertial>
+			<mass value="10"/>
+			<inertia ixx="1.0" ixy="0.0" ixz="0.0" iyy="1.0" iyz="0.0" izz="1.0"/>
+		</inertial>
 	</link>
 	<joint name="i_2" type="fixed">
-    <parent link="i1"/>
-    <child link="i2"/>
+		<parent link="i1"/>
+		<child link="i2"/>
 		<axis xyz="0 0 1"/>
-    <origin rpy = "${param['i_2']['joint_rpy']}" xyz= "${param['i_2']['joint_xyz']}"/>
-  </joint>
+		<origin rpy = "${param['i_2']['joint_rpy']}" xyz= "${param['i_2']['joint_xyz']}"/>
+	</joint>
 	<link name="i3">
 		<visual>
@@ -85,21 +85,21 @@
 			<material name="white"/>
 		</visual>
-	<collision>
+		<collision>
 			<origin rpy="0 0 0 " xyz="0.0 0 ${params['d3']/2}"/>
-      <geometry>
-        <cylinder length="${params['d3']}" radius="${params['i3_r']}"/>
-      </geometry>
-    </collision>
-    <inertial>
-      <mass value="10"/>
-      <inertia ixx="1.0" ixy="0.0" ixz="0.0" iyy="1.0" iyz="0.0" izz="1.0"/>
-    </inertial>
+			<geometry>
+				<cylinder length="${params['d3']}" radius="${params['i3_r']}"/>
+			</geometry>
+		</collision>
+		<inertial>
+			<mass value="10"/>
+			<inertia ixx="1.0" ixy="0.0" ixz="0.0" iyy="1.0" iyz="0.0" izz="1.0"/>
+		</inertial>
 	</link>
 	<joint name="i_3" type="fixed">
-    <parent link="i2"/>
-    <child link="i3"/>
+		<parent link="i2"/>
+		<child link="i3"/>
 		<axis xyz="0 0 1"/>
-    <origin rpy = "${param['i_3']['joint_rpy']}" xyz= "${param['i_3']['joint_xyz']}"/>
-  </joint>
+		<origin rpy = "${param['i_3']['joint_rpy']}" xyz= "${param['i_3']['joint_xyz']}"/>
+	</joint>
 	<link name="tool">
 		<visual>
@@ -110,19 +110,19 @@
 			<material name="blue"/>
 		</visual>
-	<collision>
+		<collision>
 			<origin rpy= "0 0 0" xyz="0.0 ${params['tool_b']/2} 0 "/>
-      <geometry>
-        <box size="${params['tool_a']} ${params['tool_b']} ${params['tool_c']}"/>
-      </geometry>
-    </collision>
-    <inertial>
-      <mass value="10"/>
-      <inertia ixx="1.0" ixy="0.0" ixz="0.0" iyy="1.0" iyz="0.0" izz="1.0"/>
-    </inertial>
+			<geometry>
+				<box size="${params['tool_a']} ${params['tool_b']} ${params['tool_c']}"/>
+			</geometry>
+		</collision>
+		<inertial>
+			<mass value="10"/>
+			<inertia ixx="1.0" ixy="0.0" ixz="0.0" iyy="1.0" iyz="0.0" izz="1.0"/>
+		</inertial>
 	</link>
 	<joint name="tool_joint" type="fixed">
-    <parent link="i3"/>
-    <child link="tool"/>
-    <origin rpy = "0.0 0.0 0.0" xyz= "0.0 0.0 ${params['d3']}"/>
-  </joint>
+		<parent link="i3"/>
+		<child link="tool"/>
+		<origin rpy = "0.0 0.0 0.0" xyz= "0.0 0.0 ${params['d3']}"/>
+	</joint>
 </robot>
