Commit message: Poprawka

File: lab_2/urdf/dynamic2.urdf.xacro (robot description, xacro)
@@ -49,6 +49,6 @@
     <parent link="base_link"/>
     <child link="i1"/>
-		<limit effort="1000.0" lower="-1.0" upper="1.0" velocity="0.5"/>
-		<axis xyz="0 1 0"/>
+		<limit effort="1000.0" lower="0" upper="1.0" velocity="0.5"/>
+		<axis xyz="0 0 1"/>
     <origin rpy = "${param['i_1']['joint_rpy']}" xyz= "0 0 ${params['base_h']}"/>
   </joint>
@@ -76,5 +76,5 @@
     <child link="i2"/>
 		<limit effort="1000.0" lower="-1.0" upper="0.0" velocity="0.5"/>
-		<axis xyz="0 1 0"/>
+		<axis xyz="0 0 1"/>
     <origin rpy = "${param['i_2']['joint_rpy']}" xyz= "${param['i_2']['joint_xyz']}"/>
   </joint>
@@ -102,5 +102,5 @@
     <child link="i3"/>
 		<limit effort="1000.0" lower="-1.0" upper="0.0" velocity="0.5"/>
-		<axis xyz="0 1 0"/>
+		<axis xyz="0 0 1"/>
     <origin rpy = "${param['i_3']['joint_rpy']}" xyz= "${param['i_3']['joint_xyz']}"/>
   </joint>
