Commit message: add KDL

File: lab_3/urdf/dynamic2.urdf.xacro (robot description, xacro)
@@ -46,5 +46,5 @@
     </inertial>
   </link>
-	<joint name="i_1" type="prismatic">
+	<joint name="i_1" type="revolute">
     <parent link="base_link"/>
     <child link="i1"/>
@@ -72,5 +72,5 @@
     </inertial>
 	</link>
-	<joint name="i_2" type="prismatic">
+	<joint name="i_2" type="revolute">
     <parent link="i1"/>
     <child link="i2"/>

Commit message: add non kdl part 2

File: lab_3/urdf/dynamic2.urdf.xacro (robot description, xacro)
@@ -51,5 +51,5 @@
 		<limit effort="1000.0" lower="0" upper="1.0" velocity="0.5"/>
 		<axis xyz="0 0 1"/>
-    <origin rpy = "${param['i_1']['joint_rpy']}" xyz= "0 0 ${params['base_h']}"/>
+    <origin rpy = "${param['i_1']['joint_rpy']}" xyz= "${param['i_1']['joint_xyz']}"/>
   </joint>
 	<link name="i2">

Commit message: add KDL and visual preferences

File: lab_3/urdf/dynamic2.urdf.xacro (robot description, xacro)
@@ -46,5 +46,5 @@
     </inertial>
   </link>
-	<joint name="i_1" type="revolute">
+	<joint name="i_1" type="prismatic">
     <parent link="base_link"/>
     <child link="i1"/>
@@ -72,5 +72,5 @@
     </inertial>
 	</link>
-	<joint name="i_2" type="revolute">
+	<joint name="i_2" type="prismatic">
     <parent link="i1"/>
     <child link="i2"/>

Commit message: fix visual part of rviz robot

File: lab_3/urdf/dynamic2.urdf.xacro (robot description, xacro)
@@ -32,5 +32,5 @@
         <box size="${params['i1_a']} ${params['i1_b']} ${params['d1']}"/>
       </geometry>
-      <origin rpy="0 0 0 " xyz="0.0 0 ${params['d1']/2}"/>
+      <origin rpy="0 0 0 " xyz="0.0 0.0 -${params['d1']/2}"/>
       <material name="blue"/>
     </visual>
@@ -58,5 +58,5 @@
 				<cylinder length="${params['d2']-params['i1_b']}" radius="${params['i2_r']}"/>
 			</geometry>
-			<origin rpy="0 0 0 " xyz="0.0 0 ${params['d2']/2}"/>
+			<origin rpy="0 0 0 " xyz="0.0 0.0 -${params['d2']/2}"/>
 			<material name="black"/>
 		</visual>
@@ -84,5 +84,5 @@
 				<cylinder length="${params['d3']-params['i2_r']}" radius=" ${params['i3_r']}"/>
 			</geometry>
-			<origin rpy="0 0 0 " xyz="0.0 0 ${params['d3']/2}"/>
+			<origin rpy="0 0 0 " xyz="0.0 0.0 -${params['d3']/2}"/>
 			<material name="white"/>
 		</visual>
@@ -127,5 +127,5 @@
     <parent link="i3"/>
     <child link="tool"/>
-    <origin rpy = "0.0 0.0 0.0" xyz= "0.0 0.0 ${params['d3']}"/>
+    <origin rpy = "0.0 0.0 0.0" xyz= "0.0 0.0 0.0"/>
   </joint>
 </robot>
